File: production/pearphone/pearphone.kicad_pcb (KiCad board)
At the start: 2 copper layers, 105 x 70.6 mm, 4 parts, among them SW1 SW_Push, U2 XIAO_ESP32C3

Commit message: Wired PCB v1 and ordered from JLC
Routing:
- net +5V: track 0.00 -> 126.7 mm
- net CTP_SDA: track 0.00 -> 126.3 mm
- net CTP_INT: track 0.00 -> 114.3 mm
- net CTP_SCL: track 0.00 -> 110.4 mm
- net CTP_RST: track 0.00 -> 107.0 mm
- net GND: track 0.00 -> 93.8 mm
- net SW1: track 0.00 -> 93.0 mm
- net MOSI: track 0.00 -> 86.0 mm
- net LCD_RS: track 0.00 -> 83.9 mm
- net MISO: track 0.00 -> 82.7 mm
- net LCD_RST: track 0.00 -> 80.4 mm
- net SCK: track 0.00 -> 79.9 mm
- net LCD_CS: track 0.00 -> 76.7 mm
